File: Hardware/backplane/jc2_backplane.kicad_sch (KiCad schematic)
At the start: 15 parts, among them J0 JC2_DIN41612_02x32_AC, J1 JC2_DIN41612_02x32_AC, J2 JC2_DIN41612_02x32_AC, J3 JC2_DIN41612_02x32_AC, J4 Flat-cable, J5 POWER

Commit message: Updates of mmu and backplane HW
Parts:
- added H1, H2, H3, H4: MountingHole, MountingHole:MountingHole_3.2mm_M3, symbol Mechanical:MountingHole
- C1, C2, C3: value 1uF -> 10 uF
- J1, J2, J3: value JC2_DIN41612_02x32_AC -> DIN41612 02x32 AC
- J4: renamed from J0; value JC2_DIN41612_02x32_AC -> DIN41612 02x32 AC
- renumbered J4 to J6
Other:
- note added: "Slot 4"
- note removed: "Slot 0"
