File: Hardware/cf_ide/jc2_cf_ide.kicad_sch (KiCad schematic)
At the start: 16 parts, among them J1 IDE-44_Header, J3 ADDR, J4 JC2_DIN41612_02x32_AC, U1 GAL16V8, U2 74LS245

Commit message: cf_ide update
Other:
- note added: "DIOW = KX & PHI2 & !A9 & !A8 & A7 & !A6 & !A5 & !A4 & !A3 & !R_W; /* $0880-$0887 write */ DIOR = KX & PHI2 & !A9 & !A8 & A7 & !A6 & !A5 & !A4 & !A3 & R_W; /* $0880-$0887 read */ RST = KX & PHI2 & !A9 & !A8 & A7 & !A6 & !A5 & !A4 & A3 & !R_W & !D0; /* $0888-$088F write 0 */ KXD = KX delayed approx. 30 nsec."
- note removed: "DIOW = KX & PHI2 & !A9 & !A8 & !A7 & !A6 & !A5 & !A4 & !A3 & !R_W; /* $0800-$0807 write */ DIOR = KX & PHI2 & !A9 & !A8 & !A7 & !A6 & !A5 & !A4 & !A3 & R_W; /* $0800-$0807 read */ RST = KX & PHI2 & !A9 & !A8 & !A7 & !A6 & !A5 & !A4 & A3 & !R_W & !D0; /* $0808-$080F write 0 */ KXD = KX delayed approx. 30 nsec."
Changed lines of the file:
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@@
 		)
 	)
-	(text "DIOW = KX & PHI2 & !A9 & !A8 & !A7 & !A6 & !A5 & !A4 & !A3 & !R_W;       /* $0800-$0807 write */\nDIOR = KX & PHI2 & !A9 & !A8 & !A7 & !A6 & !A5 & !A4 & !A3 &  R_W;       /* $0800-$0807 read */\nRST  = KX & PHI2 & !A9 & !A8 & !A7 & !A6 & !A5 & !A4 &  A3 & !R_W & !D0; /* $0808-$080F write 0 */\nKXD  = KX delayed approx. 30 nsec."
+	(text "DIOW = KX & PHI2 & !A9 & !A8 & A7 & !A6 & !A5 & !A4 & !A3 & !R_W;       /* $0880-$0887 write */\nDIOR = KX & PHI2 & !A9 & !A8 & A7 & !A6 & !A5 & !A4 & !A3 &  R_W;       /* $0880-$0887 read */\nRST  = KX & PHI2 & !A9 & !A8 & A7 & !A6 & !A5 & !A4 &  A3 & !R_W & !D0; /* $0888-$088F write 0 */\nKXD  = KX delayed approx. 30 nsec."
 		(exclude_from_sim no)
 		(at 93.472 83.312 0)
